Commit message: Update 1

File: guardrail_robot/urdf/chassis.xacro (robot description, xacro)
@@ -19,9 +19,9 @@
       </material>
     </visual>
-    <!-- Lower skirt: makes the robot look like a road-inspection platform. -->
-    <visual name="skirt_visual">
-      <origin xyz="0 0 -0.09" rpy="0 0 0"/>
+    <!-- Cabin above the main body: 4.70 m car, 1.50 m total height. -->
+    <visual name="cabin_visual">
+      <origin xyz="-0.15 0 0.55" rpy="0 0 0"/>
       <geometry>
-        <box size="0.58 0.40 0.04"/>
+        <box size="2.20 1.70 0.35"/>
       </geometry>
       <material name="body_dark">
@@ -29,9 +29,28 @@
       </material>
     </visual>
-    <!-- Front camera housing and rear equipment box are only decorative. -->
+    <!-- Lower floor pan, narrower than the track so the wheels stay visible. -->
+    <visual name="skirt_visual">
+      <origin xyz="0 0 -0.42" rpy="0 0 0"/>
+      <geometry>
+        <box size="4.30 1.30 0.15"/>
+      </geometry>
+      <material name="body_dark">
+        <color rgba="0.11 0.12 0.13 1.0"/>
+      </material>
+    </visual>
+    <!-- Front grille / bumper and rear roof equipment box are decorative. -->
     <visual name="front_panel_visual">
-      <origin xyz="0.305 0 0.01" rpy="0 0 0"/>
+      <origin xyz="2.34 0 -0.20" rpy="0 0 0"/>
       <geometry>
-        <box size="0.025 0.20 0.10"/>
+        <box size="0.06 1.50 0.30"/>
+      </geometry>
+      <material name="panel_grey">
+        <color rgba="0.20 0.22 0.24 1.0"/>
+      </material>
+    </visual>
+    <visual name="rear_box_visual">
+      <origin xyz="-0.90 0 0.835" rpy="0 0 0"/>
+      <geometry>
+        <box size="0.70 1.20 0.22"/>
       </geometry>
       <material name="panel_grey">
@@ -45,8 +64,15 @@
       </geometry>
     </collision>
+    <collision name="cabin_collision">
+      <origin xyz="-0.15 0 0.55" rpy="0 0 0"/>
+      <geometry>
+        <box size="2.20 1.70 0.35"/>
+      </geometry>
+    </collision>
+    <!-- Effective height includes the cabin and roof equipment. -->
     <xacro:box_inertial mass="${chassis_mass}"
                         x="${chassis_length}"
                         y="${chassis_width}"
-                        z="${chassis_height}"/>
+                        z="1.30"/>
   </link>
   <!-- A fixed frame at the front face, convenient for future sensors. -->
@@ -55,5 +81,5 @@
     <parent link="base_link"/>
     <child link="front_frame"/>
-    <origin xyz="0.31 0 0.02" rpy="0 0 0"/>
+    <origin xyz="2.36 0 -0.20" rpy="0 0 0"/>
   </joint>
 </robot>

File: guardrail_robot/urdf/common.xacro (robot description, xacro)
@@ -3,27 +3,34 @@
   <!-- ============================================================
        Geometric and dynamic parameters (SI units: m, kg, s, rad)
+       Real-world reference: a mid-size highway inspection car.
+       4.70 m long, 1.85 m wide, 1.50 m tall, 2.80 m wheelbase,
+       0.68 m diameter wheels.  This is proportionate to the 3.75 m
+       highway lanes in worlds/highway.sdf.
        ============================================================ -->
-  <xacro:property name="wheel_radius"     value="0.10"/>
-  <xacro:property name="wheel_width"      value="0.06"/>
-  <xacro:property name="wheel_mass"       value="0.70"/>
-  <!-- Wheel centres relative to base_link -->
-  <xacro:property name="wheel_x"          value="0.22"/>
-  <xacro:property name="wheel_y"          value="0.235"/>
-  <xacro:property name="wheel_z"          value="-0.14"/>
+  <xacro:property name="wheel_radius"     value="0.34"/>
+  <xacro:property name="wheel_width"      value="0.24"/>
+  <xacro:property name="wheel_mass"       value="25.0"/>
+  <!-- Wheel centres relative to base_link.
+       wheel_z keeps the wheel contact patch on the base_footprint plane:
+       base_link_z + wheel_z = wheel_radius. -->
+  <xacro:property name="wheel_x"          value="1.40"/>
+  <xacro:property name="wheel_y"          value="0.79"/>
+  <xacro:property name="wheel_z"          value="-0.435"/>
   <!-- Track width used by the diff-drive plugin (left/right wheel centres) -->
   <xacro:property name="wheel_separation" value="${2.0 * wheel_y}"/>
-  <!-- Chassis -->
-  <xacro:property name="chassis_length"   value="0.62"/>
-  <xacro:property name="chassis_width"    value="0.44"/>
-  <xacro:property name="chassis_height"   value="0.18"/>
-  <xacro:property name="chassis_mass"     value="8.0"/>
-  <xacro:property name="base_link_z"      value="0.24"/>
+  <!-- Body: 4.70 x 1.85 x 0.75 m (cabin adds another 0.35 m), 0.28 m
+       ground clearance under the floor pan. -->
+  <xacro:property name="chassis_length"   value="4.70"/>
+  <xacro:property name="chassis_width"    value="1.85"/>
+  <xacro:property name="chassis_height"   value="0.75"/>
+  <xacro:property name="chassis_mass"     value="1500.0"/>
+  <xacro:property name="base_link_z"      value="0.775"/>
   <!-- Sensor mounting (relative to base_link) -->
-  <xacro:property name="camera_x"         value="0.335"/>
+  <xacro:property name="camera_x"         value="2.36"/>
   <xacro:property name="camera_y"         value="0.0"/>
-  <xacro:property name="camera_z"         value="0.16"/>
+  <xacro:property name="camera_z"         value="0.025"/>
   <xacro:property name="lidar_x"          value="0.0"/>
   <xacro:property name="lidar_y"          value="0.0"/>
-  <xacro:property name="lidar_z"          value="0.22"/>
+  <xacro:property name="lidar_z"          value="0.925"/>
   <!-- ============================================================
        Inertia helpers.  All links are modelled as primitive shapes,

File: guardrail_robot/urdf/gazebo.xacro (robot description, xacro)
@@ -26,14 +26,15 @@
       <child_frame_id>base_footprint</child_frame_id>
       <odom_publish_frequency>50</odom_publish_frequency>
-      <!-- Speed and acceleration limits make the simulated vehicle
-           behave like a small inspection robot, not a racing car. -->
-      <min_linear_velocity>-1.0</min_linear_velocity>
-      <max_linear_velocity>1.5</max_linear_velocity>
+      <!-- Road-inspection vehicle limits: up to 10 m/s (36 km/h) and
+           3 m/s^2 acceleration, i.e. quick enough to drive normally on
+           the 120 m highway section while staying controllable. -->
+      <min_linear_velocity>-4.0</min_linear_velocity>
+      <max_linear_velocity>10.0</max_linear_velocity>
       <min_angular_velocity>-2.0</min_angular_velocity>
       <max_angular_velocity>2.0</max_angular_velocity>
-      <min_linear_acceleration>-1.0</min_linear_acceleration>
-      <max_linear_acceleration>1.0</max_linear_acceleration>
-      <min_angular_acceleration>-2.0</min_angular_acceleration>
-      <max_angular_acceleration>2.0</max_angular_acceleration>
+      <min_linear_acceleration>-5.0</min_linear_acceleration>
+      <max_linear_acceleration>3.0</max_linear_acceleration>
+      <min_angular_acceleration>-3.0</min_angular_acceleration>
+      <max_angular_acceleration>3.0</max_angular_acceleration>
     </plugin>
     <!-- Publishes /joint_states as gz.msgs.Model; bridge it to

File: guardrail_robot/urdf/sensors.xacro (robot description, xacro)
@@ -6,5 +6,5 @@
       <origin xyz="0 0 0" rpy="0 0 0"/>
       <geometry>
-        <box size="0.050 0.090 0.055"/>
+        <box size="0.075 0.135 0.080"/>
       </geometry>
       <material name="sensor_dark">
@@ -13,7 +13,7 @@
     </visual>
     <visual name="camera_lens_visual">
-      <origin xyz="0.028 0 0" rpy="0 1.5708 0"/>
+      <origin xyz="0.042 0 0" rpy="0 1.5708 0"/>
       <geometry>
-        <cylinder radius="0.018" length="0.012"/>
+        <cylinder radius="0.027" length="0.018"/>
       </geometry>
       <material name="lens_blue">
@@ -23,7 +23,7 @@
     <!-- Small bracket down to the chassis front face. -->
     <visual name="camera_bracket_visual">
-      <origin xyz="-0.020 0 -0.045" rpy="0 0 0"/>
+      <origin xyz="-0.020 0 -0.060" rpy="0 0 0"/>
       <geometry>
-        <box size="0.030 0.040 0.090"/>
+        <box size="0.040 0.060 0.120"/>
       </geometry>
       <material name="panel_grey">
@@ -34,8 +34,8 @@
       <origin xyz="0 0 0" rpy="0 0 0"/>
       <geometry>
-        <box size="0.050 0.090 0.055"/>
+        <box size="0.075 0.135 0.080"/>
       </geometry>
     </collision>
-    <xacro:box_inertial mass="0.15" x="0.050" y="0.090" z="0.055"/>
+    <xacro:box_inertial mass="0.30" x="0.075" y="0.135" z="0.080"/>
   </link>
   <joint name="camera_joint" type="fixed">
@@ -77,7 +77,7 @@
     <!-- Mounting mast -->
     <visual name="lidar_mast_visual">
-      <origin xyz="0 0 -0.055" rpy="0 0 0"/>
+      <origin xyz="0 0 -0.100" rpy="0 0 0"/>
       <geometry>
-        <cylinder radius="0.022" length="0.110"/>
+        <cylinder radius="0.030" length="0.200"/>
       </geometry>
       <material name="panel_grey">
@@ -109,5 +109,5 @@
       </geometry>
     </collision>
-    <xacro:cylinder_inertial mass="0.25" radius="0.055" length="0.060"/>
+    <xacro:cylinder_inertial mass="0.80" radius="0.055" length="0.060"/>
   </link>
   <joint name="lidar_joint" type="fixed">
@@ -131,5 +131,5 @@
            Otherwise the lens/body can clip into the camera's near plane and
            fill the whole image with its own housing. -->
-      <pose>0.06 0 0 0 0 0</pose>
+      <pose>0.09 0 0 0 0 0</pose>
       <camera>
         <horizontal_fov>1.396263</horizontal_fov>

File: guardrail_robot/urdf/wheels.xacro (robot description, xacro)
@@ -18,5 +18,5 @@
         <origin xyz="0 0 0" rpy="${pi/2} 0 0"/>
         <geometry>
-          <cylinder radius="${0.055}" length="${wheel_width + 0.004}"/>
+          <cylinder radius="${0.22}" length="${wheel_width + 0.004}"/>
         </geometry>
         <material name="rim_silver">
@@ -24,5 +24,9 @@
         </material>
       </visual>
-      <collision name="${name}_tyre_collision">
+      <!-- The collision name must start with the link name (or be empty).
+           Otherwise sdformat prefixes it with "fixed_joint_lump" and silently
+           drops the <gazebo> friction extension below, leaving the wheels at
+           the default friction. -->
+      <collision name="${name}_wheel_link_tyre_collision">
         <origin xyz="0 0 0" rpy="${pi/2} 0 0"/>
         <geometry>
@@ -39,13 +43,19 @@
       <origin xyz="${x} ${y} ${wheel_z}" rpy="0 0 0"/>
       <axis xyz="0 1 0"/>
-      <limit effort="20.0" velocity="30.0"/>
+      <!-- Car-sized wheel: about 136 Nm per wheel for 1 m/s^2, with a large
+           reserve for scrubbing the tyres during skid-steer turns. -->
+      <limit effort="1500.0" velocity="60.0"/>
       <dynamics damping="0.05" friction="0.0"/>
     </joint>
-    <!-- High friction is needed for skid-steer / four-wheel differential drive.
-         The values are Gazebo URDF extensions and are converted to SDF surface
-         parameters when the robot is spawned. -->
+    <!-- Skid-steer friction: mu1 is the longitudinal tread grip, mu2 is the
+         lateral scrub.  Keeping mu2 well below mu1 lets the four non-steered
+         wheels slide sideways when the differential drive rotates the car.
+         With mu1 == mu2 the long 2.8 m wheelbase cannot overcome the lateral
+         friction and the car barely turns.  fdir1 keeps mu1 along the rolling
+         direction (wheel link +x). -->
     <gazebo reference="${name}_wheel_link">
-      <mu1>1.2</mu1>
-      <mu2>1.2</mu2>
+      <mu1>1.5</mu1>
+      <mu2>0.2</mu2>
+      <fdir1>1 0 0</fdir1>
       <kp>1000000.0</kp>
       <kd>100.0</kd>
